File: KiCad/GR_LDO_Distribution.kicad_pcb (KiCad board)
At the start: 2 copper layers, 64.8 x 56.5 mm, 66 parts, among them J1 Screw_Terminal_01x02, J10 Conn_01x02, J11 Conn_01x02, J12 Conn_01x02, J13 Conn_01x02, J2 Conn_01x03, J3 Conn_01x04, J4 Conn_01x02, J5 Conn_01x02, J6 Conn_01x02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

Commit message: Add files via upload
Parts:
- removed J11, J13, J9: Conn_01x02, Connector_JST:JST_XH_B2B-XH-A_1x02_P2.50mm_Vertical
- removed the J5 at (142.6, 125.1)
- removed the J6 at (152.0, 125.0)
- removed the J7 at (161.4, 125.1)
- R10, R12, R4, R6, R8: value 1K3 -> 1K2
- R11, R3, R5, R7, R9: value 240r -> 220r
- moved J4 23.4 mm to (156.5, 125.0)
- moved J6 4.80 mm to (134.4, 74.5)
- moved J7 4.50 mm to (115.8, 74.5)
- moved J5 4.00 mm to (153.8, 74.4)
- renumbered J8 to J5, J10 to J6, J12 to J7
Connections:
- C1 pad 1: /Vin -> /5VIn
- F2 pad 1: Net-(F2-Pad1) -> /5VIn
- J4 pad 1: Net-(F2-Pad1) -> Net-(F3-Pad1)
- TP2 pad 1: Net-(F2-Pad1) -> /5VIn
- U1 pad 3: /Vin -> /5VIn
Routing:
- net Net-(F2-Pad1): track 24.4 -> 0.00 mm
- net /5VIn: track 0.00 -> 20.8 mm
- net /Vin: track 166.1 -> 149.4 mm
- net Net-(F5-Pad1): track 24.5 -> 12.6 mm
- net Net-(F4-Pad1): track 24.5 -> 12.6 mm
- net Net-(F3-Pad1): track 24.9 -> 13.0 mm
- net Net-(F6-Pad1): track 24.2 -> 12.5 mm
- net GNDREF: track 16.7 -> 11.4 mm, vias 25 -> 16
- net Net-(C3-Pad1): vias 10 -> 20
- net Net-(C14-Pad1): vias 14 -> 24
